File: hardware/prototype.kicad_pcb (KiCad board)
At the start: 2 copper layers, 102.5 x 66.1 mm, 53 parts, among them J1 ANT, J2 Micro USB, J3 IGC, U1 LM2936-3.3, Y1 12M

Commit message: Unfinished pcb layouts
Parts:
- C13, C14: footprint Capacitors_ThroughHole:C_Disc_D5.0mm_W2.5mm_P5.00mm -> Capacitors_SMD:C_0603_HandSoldering
- F1: footprint Fuse_Holders_and_Fuses:Fuse_SMD1206_Reflow -> Fuse_Holders_and_Fuses:Fuse_TE5_Littlefuse-395Series
- moved F1 18.7 mm to (196.0, 94.3), turned to 270 degrees
- moved C13 0.83 mm to (183.2, 111.6), turned to 0 degrees
- moved C14 0.38 mm to (183.3, 114.1), turned to 0 degrees
Routing:
- net 3.3V: track 294.5 -> 314.9 mm
- net 5V: track 79.9 -> 67.7 mm, vias 3 -> 2
- net /Console/USB_5V: track 7.95 -> 15.5 mm, vias 0 -> 1
- net /SPI_CLOCK: track 41.8 -> 46.1 mm
- net /CHIP_RESET: track 57.9 -> 60.5 mm
- net Earth: track 35.1 -> 37.6 mm
- net /BARO_SCL: track 31.9 -> 34.4 mm
- net /BARO_SDA: track 30.1 -> 32.1 mm
- net /AUX_STATUS: track 55.4 -> 54.0 mm
- net /Console/USB_D-: track 20.6 -> 21.7 mm
- net /GPS_ENABLE: track 23.1 -> 24.1 mm
- net /SPI_MISO: track 36.4 -> 37.5 mm
- net /SD_CS: track 86.7 -> 85.7 mm
- net /Console/RS232_RX: track 22.5 -> 23.2 mm
- net /SPI_SELECT: track 25.1 -> 25.7 mm
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Other:
- net class ANT: via_drill 0.3 -> 0.5
- net class Default: via_dia 1 -> 1.5; via_drill 0.3 -> 0.5
- net class HV: via_dia 1.2 -> 1.8; via_drill 0.3 -> 0.5
- net class PWR: via_dia 1 -> 1.5; via_drill 0.3 -> 0.5
- net class USB added: clearance 0.2, trace_width 0.3, via_dia 1.5, via_drill 0.5
