File: hardware/ogntracker.sch (KiCad schematic (older format))
At the start: 13 parts, among them J1 ANT, J2 CONN_PWR, U1 STM32DEVBOARD, U2 RFM69HW, U3 VK2828U7G5LF

Commit message: Improvements to make hand-made board easier to produce
 * Wider copper base for pins
 * Proper size of CPU board
 * Added console headers
Parts:
- added UART1: CONSOLE1, symbol CONN_01X04
- added UART2: CONSOLE2, symbol CONN_01X04
- C1, C3, C4: footprint Capacitors_ThroughHole:C_Rect_L7_W2.5_P5 -> OGN Tracker:C_Rect_L7_W2.5_P5
- C2, C5: footprint Capacitors_ThroughHole:C_Radial_D5_L11_P2.5 -> OGN Tracker:C_Radial_D5_L11_P2.5
- D1: footprint Connectors_Molex:Molex_PicoBlade_53047-0210_02x1.25mm_Straight -> OGN Tracker:Molex_PicoBlade_53047-0210_02x1.25mm_Straight
- J2: footprint Kedder Terminals:XY301-5-2 -> OGN Tracker:XY301-5-2
- R1: footprint Resistors_ThroughHole:Resistor_Horizontal_RM7mm -> OGN Tracker:Resistor_Horizontal_RM7mm
- U3: footprint Connectors_Molex:Molex_PicoBlade_53047-0610_06x1.25mm_Straight -> OGN Tracker:Molex_PicoBlade_53047-0610_06x1.25mm_Straight
- renumbered PWR1 to SUP1
Connections:
- net labels added: ANT, CON1_RXD, CON1_TXD, CON2_RXD, CON2_TXD, LED
- wire segments 58 -> 70

Commit message: Version 0.2.0, manufactured
Parts:
- UART1, UART2: footprint (none) -> Pin_Headers:Pin_Header_Straight_1x04
Changed lines of the file:
@@
 F 0 "UART1" H 7350 4450 50  0000 C CNN
 F 1 "CONSOLE1" V 7450 4200 50  0000 C CNN
-F 2 "" H 7350 4200 50  0001 C CNN
+F 2 "Pin_Headers:Pin_Header_Straight_1x04" H 7350 4200 50  0001 C CNN
 F 3 "" H 7350 4200 50  0001 C CNN
 	1    7350 4200
@@
 $EndComp
 $Comp
-L Earth #PWR?
+L Earth #PWR011
 U 1 1 59A1BB3D
 P 7050 3950
-F 0 "#PWR?" H 7050 3700 50  0001 C CNN
+F 0 "#PWR011" H 7050 3700 50  0001 C CNN
 F 1 "Earth" H 7050 3800 50  0001 C CNN
 F 2 "" H 7050 3950 50  0001 C CNN
@@
 F 0 "UART2" H 3250 5450 50  0000 C CNN
 F 1 "CONSOLE2" V 3350 5200 50  0000 C CNN
-F 2 "" H 3250 5200 50  0001 C CNN
+F 2 "Pin_Headers:Pin_Header_Straight_1x04" H 3250 5200 50  0001 C CNN
 F 3 "" H 3250 5200 50  0001 C CNN
 	1    3250 5200
@@
 $EndComp
 $Comp
-L Earth #PWR?
+L Earth #PWR012
 U 1 1 59A1C116
 P 3550 5450
-F 0 "#PWR?" H 3550 5200 50  0001 C CNN
+F 0 "#PWR012" H 3550 5200 50  0001 C CNN
 F 1 "Earth" H 3550 5300 50  0001 C CNN
 F 2 "" H 3550 5450 50  0001 C CNN

Commit message: MAX232 added and 2 RJ45 sockets for comms
Parts:
- removed J2: CONN_PWR, OGN Tracker:XY301-5-2, symbol CONN_01X02
- removed UART1: CONSOLE1, Pin_Headers:Pin_Header_Straight_1x04, symbol CONN_01X04
- removed UART2: CONSOLE2, Pin_Headers:Pin_Header_Straight_1x04, symbol CONN_01X04
- added C? (x5): 1uF, symbol C_Small
- added J?: IGC, symbol RJ45
- added J?: LX, symbol RJ45
- added U?: MAX232, symbol MAX232
Connections:
- net labels added: RS232_RX, RS232_TX
- net labels removed: CON2_RXD, CON2_TXD
- wire segments 70 -> 106
Other:
- moved on the sheet: C1, C3, C4, D1, J1, R1, U2, U3

Commit message: Hardware 0.3 released for manufacturing
Parts:
- removed C2: 1uF, OGN Tracker:C_Radial_D5_L11_P2.5, symbol CP_Small
- removed C5: 10uF, OGN Tracker:C_Radial_D5_L11_P2.5, symbol CP_Small
- removed SUP1: BUCK_CONVERTER, OGN Tracker:Buck_Converter_Sm, symbol BUCK_CONVERTER
- added BARO1: BMP280, OGN Tracker:BMP280, symbol BMP280
- added C11: 100nF, Capacitors_SMD:C_1206_HandSoldering, symbol C_Small
- added C2: 1uF, Capacitors_SMD:C_1206_HandSoldering, symbol C_Small
- added C5: 330uF, Capacitors_ThroughHole:C_Radial_D8_L13_P3.8, symbol CP1
- added D2: 1N4001, Diodes_ThroughHole:Diode_DO-35_SOD27_Horizontal_RM10, symbol D
- added L1: 1uH, Inductors:INDUCTOR_V, symbol Ferrite_Bead
- added R2, R3: 10K, Resistors_SMD:R_1206_HandSoldering, symbol R
- added SUP1: BUCK_CVTR, OGN Tracker:Buck_Converter_Sm, symbol BUCK_CVTR
- C1, C3: footprint OGN Tracker:C_Rect_L7_W2.5_P5 -> Capacitors_SMD:C_1206_HandSoldering
- C10, C6, C7, C8, C9: renamed from C?; footprint (none) -> Capacitors_SMD:C_1206_HandSoldering
- C4: value 100nF -> 1uF; footprint OGN Tracker:C_Rect_L7_W2.5_P5 -> Capacitors_SMD:C_1206_HandSoldering
- J2, J3: renamed from J?; footprint (none) -> OGN Tracker:RJ45_SOCKET_SHLD
- R1: value R -> 330; footprint OGN Tracker:Resistor_Horizontal_RM7mm -> Resistors_SMD:R_1206_HandSoldering
- U4: renamed from U?; footprint (none) -> OGN Tracker:DIP-16_W7.62mm
Connections:
- net labels added: BARO_SCL, BARO_SDA, RP_PROTECTION, SUP_CLEAN
- wire segments 106 -> 126
- no-connect marks 0 -> 1
Other:
- moved on the sheet: C4

Commit message: Various updates to schematics and experiments with layout for new box
Parts:
- added C12: 100nF, Capacitors_SMD:C_1206, symbol C_Small
- added D3, D4: 1N4148, symbol D_Small
- added R4, R5: 10K, symbol R_Small
- added U5: SDCARD_SPI, Connect:SD_Card_Receptacle, symbol SDCARD_SPI
- C1, C11, C2, C3, C4: footprint Capacitors_SMD:C_1206_HandSoldering -> Capacitors_SMD:C_1206
- C10, C6, C7, C8, C9: footprint Capacitors_SMD:C_1206_HandSoldering -> Capacitors_SMD:C_0805
- R1: value 330 -> 90; footprint Resistors_SMD:R_1206_HandSoldering -> Resistors_SMD:R_1206
- R2, R3: footprint Resistors_SMD:R_1206_HandSoldering -> Resistors_SMD:R_1206
- U4: footprint OGN Tracker:DIP-16_W7.62mm -> Housings_SOIC:SOIC-16_3.9x9.9mm_Pitch1.27mm
Connections:
- net labels added: SD_CS, SD_MISO, SD_MOSI, SD_SCK
- wire segments 126 -> 153
Other:
- moved on the sheet: C10, C6, C7, C8, C9, J2, J3, U4

Commit message: Routed prototype board for HAMMOND 1593N box
Parts:
- removed C10, C6, C7, C8, C9: 1uF, Capacitors_SMD:C_0805, symbol C_Small
- removed D3, D4: 1N4148, symbol D_Small
- removed J2: LX, OGN Tracker:RJ45_SOCKET_SHLD, symbol RJ45
- removed J3: IGC, OGN Tracker:RJ45_SOCKET_SHLD, symbol RJ45
- removed R4, R5: 10K, symbol R_Small
- removed U4: MAX232, Housings_SOIC:SOIC-16_3.9x9.9mm_Pitch1.27mm, symbol MAX232
- removed U5: SDCARD_SPI, Connect:SD_Card_Receptacle, symbol SDCARD_SPI
- added C15: 47uF, Capacitors_SMD:C_1210, symbol C_Small
- added C16: 1uF, Capacitors_SMD:C_1206, symbol C_Small
- added D6: LED_BT, OGN Tracker:Molex_PicoBlade_02x1.25mm_HandSoldering, symbol LED
- added LS1: Buzzer, Buzzers_Beepers:Buzzer_12x9.5RM7.6, symbol Speaker
- added R10: 82, Resistors_SMD:R_1206, symbol R_Small
- added R7, R8, R9: 10K, Resistors_SMD:R_1206, symbol R_Small
- added SDCARD1: Micro SD Reader, OGN Tracker:SDCARD_BOMB, symbol Micro_SD_Card_Det1
- added U1: LM2936-3.3, TO_SOT_Packages_SMD:SOT-223-3Lead_TabPin2, symbol LM2936-3.3
- BARO1: footprint OGN Tracker:BMP280 -> OGN Tracker:BMP280_HandSoldering
- D1: value LED -> LED_STAT; footprint OGN Tracker:Molex_PicoBlade_53047-0210_02x1.25mm_Straight -> OGN Tracker:Molex_PicoBlade_02x1.25mm_HandSoldering
- GPS1: renamed from U3; footprint OGN Tracker:Molex_PicoBlade_53047-0610_06x1.25mm_Straight -> OGN Tracker:Molex_PicoBlade_06x1.25mm_HandSoldering
- PWR1: renamed from SUP1; footprint OGN Tracker:Buck_Converter_Sm -> OGN Tracker:Buck_Converter_Sm_HandSoldering
- R1: value 90 -> 82
- STM32: renamed from U1; footprint OGN Tracker:STM32DEVBOARD -> OGN Tracker:STM32DEVBOARD_HandSoldering
- renumbered U2 to RFM69HW1
Connections:
- net labels added: BUZ_IN, BUZ_OUT
- net labels removed: RS232_RX, RS232_TX
- wire segments 153 -> 126
Other:
- moved on the sheet: C4

Commit message: STM32 dev-board based schematics
Parts:
- added F1, F2: 0.5A, Fuse_Holders_and_Fuses:Fuse_SMD1206_Reflow, symbol Polyfuse_Small
- C5: footprint Capacitors_ThroughHole:C_Radial_D8_L13_P3.8 -> Capacitors_ThroughHole:CP_Radial_D8.0mm_P3.80mm
- D2: footprint Diodes_ThroughHole:Diode_DO-35_SOD27_Horizontal_RM10 -> Diodes_SMD:D_SMA_Standard
- GPS1: footprint OGN Tracker:Molex_PicoBlade_06x1.25mm_HandSoldering -> Pin_Headers:Pin_Header_Straight_1x06_Pitch2.00mm
Connections:
- net labels added: 5V_PROT, SUP_PROT
- wire segments 126 -> 129
Other:
- moved on the sheet: C1, C15, C16, U1
Changed lines of the file:
@@
 F 0 "GPS1" H 2100 4900 40  0000 L CNN
 F 1 "VK2828U7G5LF" H 2550 4150 40  0000 C CNN
-F 2 "OGN Tracker:Molex_PicoBlade_06x1.25mm_HandSoldering" H 3000 4600 40  0001 C CNN
+F 2 "Pin_Headers:Pin_Header_Straight_1x06_Pitch2.00mm" H 3000 4600 40  0001 C CNN
 F 3 "" H 3000 4600 40  0001 C CNN
 	1    2550 4400
 	1    0    0    -1
 $EndComp
-Text GLabel 2700 3850 1    60   Input ~ 0
-5V
 Text Label 3200 3600 0    40   ~ 0
 GPS_RXD
@@
 L Earth #PWR04
 U 1 1 5983759C
+P 3200 3850
+F 0 "#PWR04" H 3200 3600 50  0001 C CNN
+F 1 "Earth" H 3200 3700 50  0001 C CNN
+F 2 "" H 3200 3850 50  0001 C CNN
+F 3 "" H 3200 3850 50  0001 C CNN
+	1    3200 3850
+	0    -1   -1   0
+$EndComp
+$Comp
+L C_Small C1
+U 1 1 598375E1
 P 3100 3850
-F 0 "#PWR04" H 3100 3600 50  0001 C CNN
-F 1 "Earth" H 3100 3700 50  0001 C CNN
-F 2 "" H 3100 3850 50  0001 C CNN
+F 0 "C1" H 3110 3920 50  0000 L CNN
+F 1 "100nF" H 3110 3770 50  0000 L CNN
+F 2 "Capacitors_SMD:C_1206" H 3100 3850 50  0001 C CNN
 F 3 "" H 3100 3850 50  0001 C CNN
 	1    3100 3850
-	0    -1   -1   0
-$EndComp
-$Comp
-L C_Small C1
-U 1 1 598375E1
-P 3000 3850
-F 0 "C1" H 3010 3920 50  0000 L CNN
-F 1 "100nF" H 3010 3770 50  0000 L CNN
-F 2 "Capacitors_SMD:C_1206" H 3000 3850 50  0001 C CNN
-F 3 "" H 3000 3850 50  0001 C CNN
-	1    3000 3850
 	0    -1   -1   0
 $EndComp
@@
 L +12V #PWR07
 U 1 1 59838C1F
-P 850 1800
-F 0 "#PWR07" H 850 1650 50  0001 C CNN
-F 1 "+12V" H 850 1940 50  0000 C CNN
-F 2 "" H 850 1800 50  0001 C CNN
-F 3 "" H 850 1800 50  0001 C CNN
-	1    850  1800
-	1    0    0    -1
-$EndComp
-Text GLabel 2650 2050 1    60   Input ~ 0
+P 850 1500
+F 0 "#PWR07" H 850 1350 50  0001 C CNN
+F 1 "+12V" H 850 1640 50  0000 C CNN
+F 2 "" H 850 1500 50  0001 C CNN
+F 3 "" H 850 1500 50  0001 C CNN
+	1    850  1500
+	1    0    0    -1
+$EndComp
+Text GLabel 2650 1800 1    60   Input ~ 0
 5V
 Text GLabel 4100 4600 0    60   Input ~ 0
@@
 	5200 6150 5800 6150
 Wire Wire Line
-	2700 3850 2900 3850
+	2700 3850 3000 3850
 Wire Wire Line
 	2700 3900 2700 3850
@@
 F 0 "D2" H 850 2300 50  0000 C CNN
 F 1 "1N4001" H 850 2100 50  0000 C CNN
-F 2 "Diodes_ThroughHole:Diode_DO-35_SOD27_Horizontal_RM10" H 850 2200 50  0001 C CNN
+F 2 "Diodes_SMD:D_SMA_Standard" H 850 2200 50  0001 C CNN
 F 3 "" H 850 2200 50  0001 C CNN
 	1    850  2200
@@
 F 0 "C5" H 1375 1650 50  0000 L CNN
 F 1 "330uF" H 1375 1450 50  0000 L CNN
-F 2 "Capacitors_ThroughHole:C_Radial_D8_L13_P3.8" H 1350 1550 50  0001 C CNN
+F 2 "Capacitors_ThroughHole:CP_Radial_D8.0mm_P3.80mm" H 1350 1550 50  0001 C CNN
 F 3 "" H 1350 1550 50  0001 C CNN
 	1    1350 1550
@@
 BUZ_IN
 Wire Wire Line
-	4450 4600 4100 4600
+	4100 4600 4450 4600
 Wire Wire Line
 	4200 4600 4200 4700
@@
 Connection ~ 4350 4900
 Wire Wire Line
-	2550 2050 2800 2050
+	2550 2050 2700 2050
 $Comp
 L Earth #PWR016
 U 1 1 5A023604
-P 3100 2450
-F 0 "#PWR016" H 3100 2200 50  0001 C CNN
-F 1 "Earth" H 3100 2300 50  0001 C CNN
-F 2 "" H 3100 2450 50  0001 C CNN
-F 3 "" H 3100 2450 50  0001 C CNN
-	1    3100 2450
-	1    0    0    -1
-$EndComp
-Wire Wire Line
-	3100 2350 3100 2450
-Wire Wire Line
-	3400 2050 3550 2050
-Text GLabel 3550 2050 2    60   Input ~ 0
+P 3400 2450
+F 0 "#PWR016" H 3400 2200 50  0001 C CNN
+F 1 "Earth" H 3400 2300 50  0001 C CNN
+F 2 "" H 3400 2450 50  0001 C CNN
+F 3 "" H 3400 2450 50  0001 C CNN
+	1    3400 2450
+	1    0    0    -1
+$EndComp
+Wire Wire Line
+	3400 2350 3400 2450
+Wire Wire Line
+	3700 2050 3850 2050
+Text GLabel 3850 2050 2    60   Input ~ 0
 3.3V
 $Comp
 L C_Small C15
 U 1 1 5A02380C
-P 3450 2250
-F 0 "C15" H 3460 2320 50  0000 L CNN
-F 1 "47uF" H 3460 2170 50  0000 L CNN
-F 2 "Capacitors_SMD:C_1210" H 3450 2250 50  0001 C CNN
-F 3 "" H 3450 2250 50  0001 C CNN
-	1    3450 2250
-	1    0    0    -1
-$EndComp
-Wire Wire Line
-	3450 2050 3450 2150
-Connection ~ 3450 2050
+P 3750 2250
+F 0 "C15" H 3760 2320 50  0000 L CNN
+F 1 "47uF" H 3760 2170 50  0000 L CNN
+F 2 "Capacitors_SMD:C_1210" H 3750 2250 50  0001 C CNN
+F 3 "" H 3750 2250 50  0001 C CNN
+	1    3750 2250
+	1    0    0    -1
+$EndComp
+Wire Wire Line
+	3750 2050 3750 2150
+Connection ~ 3750 2050
 $Comp
 L Earth #PWR017
 U 1 1 5A023990
-P 3450 2450
-F 0 "#PWR017" H 3450 2200 50  0001 C CNN
-F 1 "Earth" H 3450 2300 50  0001 C CNN
-F 2 "" H 3450 2450 50  0001 C CNN
-F 3 "" H 3450 2450 50  0001 C CNN
-	1    3450 2450
-	1    0    0    -1
-$EndComp
-Wire Wire Line
-	3450 2350 3450 2450
+P 3750 2450
+F 0 "#PWR017" H 3750 2200 50  0001 C CNN
+F 1 "Earth" H 3750 2300 50  0001 C CNN
+F 2 "" H 3750 2450 50  0001 C CNN
+F 3 "" H 3750 2450 50  0001 C CNN
+	1    3750 2450
+	1    0    0    -1
+$EndComp
+Wire Wire Line
+	3750 2350 3750 2450
 $Comp
 L C_Small C16
 U 1 1 5A024206
-P 2650 2250
-F 0 "C16" H 2660 2320 50  0000 L CNN
-F 1 "1uF" H 2660 2170 50  0000 L CNN
-F 2 "Capacitors_SMD:C_1206" H 2650 2250 50  0001 C CNN
-F 3 "" H 2650 2250 50  0001 C CNN
-	1    2650 2250
+P 3000 2250
+F 0 "C16" H 3010 2320 50  0000 L CNN
+F 1 "1uF" H 3010 2170 50  0000 L CNN
+F 2 "Capacitors_SMD:C_1206" H 3000 2250 50  0001 C CNN
+F 3 "" H 3000 2250 50  0001 C CNN
+	1    3000 2250
 	1    0    0    -1
 $EndComp
@@
 L Earth #PWR018
 U 1 1 5A0243BD
-P 2650 2450
-F 0 "#PWR018" H 2650 2200 50  0001 C CNN
-F 1 "Earth" H 2650 2300 50  0001 C CNN
-F 2 "" H 2650 2450 50  0001 C CNN
-F 3 "" H 2650 2450 50  0001 C CNN
-	1    2650 2450
-	1    0    0    -1
-$EndComp
-Wire Wire Line
-	2650 2350 2650 2450
-Wire Wire Line
-	2650 2150 2650 2050
+P 3000 2450
+F 0 "#PWR018" H 3000 2200 50  0001 C CNN
+F 1 "Earth" H 3000 2300 50  0001 C CNN
+F 2 "" H 3000 2450 50  0001 C CNN
+F 3 "" H 3000 2450 50  0001 C CNN
+	1    3000 2450
+	1    0    0    -1
+$EndComp
+Wire Wire Line
+	3000 2350 3000 2450
 Connection ~ 2650 2050
 $Comp
 L LM2936-3.3 U1
 U 1 1 5A02514F
-P 3100 2050
-F 0 "U1" H 2950 2175 50  0000 C CNN
-F 1 "LM2936-3.3" H 3100 2175 50  0000 L CNN
-F 2 "TO_SOT_Packages_SMD:SOT-223-3Lead_TabPin2" H 3100 2275 50  0001 C CIN
-F 3 "" H 3100 2000 50  0001 C CNN
-	1    3100 2050
-	1    0    0    -1
-$EndComp
+P 3400 2050
+F 0 "U1" H 3250 2175 50  0000 C CNN
+F 1 "LM2936-3.3" H 3400 2175 50  0000 L CNN
+F 2 "TO_SOT_Packages_SMD:SOT-223-3Lead_TabPin2" H 3400 2275 50  0001 C CIN
+F 3 "" H 3400 2000 50  0001 C CNN
+	1    3400 2050
+	1    0    0    -1
+$EndComp
+$Comp
+L Polyfuse_Small F1
+U 1 1 5A148D8E
+P 850 1700
+F 0 "F1" V 775 1700 50  0000 C CNN
+F 1 "0.5A" V 925 1700 50  0000 C CNN
+F 2 "Fuse_Holders_and_Fuses:Fuse_SMD1206_Reflow" H 900 1500 50  0001 L CNN
+F 3 "" H 850 1700 50  0001 C CNN
+	1    850  1700
+	1    0    0    -1
+$EndComp
+Wire Wire Line
+	850  1500 850  1600
+$Comp
+L Polyfuse_Small F2
+U 1 1 5A1493BC
+P 2800 2050
+F 0 "F2" V 2725 2050 50  0000 C CNN
+F 1 "0.5A" V 2875 2050 50  0000 C CNN
+F 2 "Fuse_Holders_and_Fuses:Fuse_SMD1206_Reflow" H 2850 1850 50  0001 L CNN
+F 3 "" H 2800 2050 50  0001 C CNN
+	1    2800 2050
+	0    1    1    0
+$EndComp
+Wire Wire Line
+	2900 2050 3100 2050
+Wire Wire Line
+	3000 2150 3000 2050
+Connection ~ 3000 2050
+Wire Wire Line
+	2650 1800 2650 2050
+Text Label 900  1950 0    40   ~ 0
+SUP_PROT
+Text Label 2900 2050 0    40   ~ 0
+5V_PROT
+Text Label 2700 3850 0    40   ~ 0
+5V_PROT
 $EndSCHEMATC

Commit message: Unverified attempt on standalone STM32 chip
Parts:
- removed C4: 1uF, Capacitors_SMD:C_1206, symbol C_Small
- removed D1: LED_STAT, OGN Tracker:Molex_PicoBlade_02x1.25mm_HandSoldering, symbol LED
- removed R1: 82, Resistors_SMD:R_1206, symbol R
- removed STM32: STM32DEVBOARD, OGN Tracker:STM32DEVBOARD_HandSoldering, symbol STM32DEVBOARD
- added C10, C11, C18, C8, C9: 100nF, Capacitors_SMD:C_0805, symbol C_Small
- added C12, C13, C14, C15: 22pF, Capacitors_SMD:C_0603_HandSoldering, symbol C_Small
- added C17: 1uF, Capacitors_SMD:C_1206, symbol C_Small
- added CPU1: STM32F103, Housings_QFP:LQFP-48_7x7mm_Pitch0.5mm, symbol STM32F103
- added D2: STATUS_PANEL, OGN Tracker:Molex_PicoBlade_02x1.25mm_HandSoldering, symbol LED_Small
- added D3: STATUS_SMD, LEDs:LED_0603, symbol LED_Small
- added D4: PWR, LEDs:LED_0603, symbol LED_Small
- added J2: SWD, Pin_Headers:Pin_Header_Straight_1x04_Pitch2.54mm, symbol CONN_01X04
- added J3: BOOT, Pin_Headers:Pin_Header_Straight_2x03_Pitch2.54mm, symbol CONN_02X03
- added R1: 82, Resistors_SMD:R_0805, symbol R_Small
- added R11, R12, R13: 10K, Resistors_SMD:R_0805, symbol R_Small
- added R2, R3: 330, Resistors_SMD:R_0805, symbol R_Small
- added R8: 1M, Resistors_SMD:R_0805, symbol R_Small
- added SW1: RESET, Buttons_Switches_SMD:SW_SPST_REED_CT05-XXXX-G1, symbol SW_Push
- added Y1: 32.768K, Crystals:Crystal_SMD_SeikoEpson_MC306-4pin_8.0x3.2mm, symbol Crystal_GND23_Small
- added Y2: 8MHz, Crystals:Crystal_HC49-4H_Vertical, symbol Crystal_Small
- C16: renamed from C11; footprint Capacitors_SMD:C_1206 -> Capacitors_SMD:C_0805
- C2: renamed from C1; footprint Capacitors_SMD:C_1206 -> Capacitors_SMD:C_0805
- C4: renamed from C3; footprint Capacitors_SMD:C_1206 -> Capacitors_SMD:C_0805
- C7: renamed from C12; footprint Capacitors_SMD:C_1206 -> Capacitors_SMD:C_0805
- R10: renamed from R3; footprint Resistors_SMD:R_1206 -> Resistors_SMD:R_0805
- R4: renamed from R7; footprint Resistors_SMD:R_1206 -> Resistors_SMD:R_0805
- R5: renamed from R8; footprint Resistors_SMD:R_1206 -> Resistors_SMD:R_0805
- R6: renamed from R9; footprint Resistors_SMD:R_1206 -> Resistors_SMD:R_0805
- R7: renamed from R10; footprint Resistors_SMD:R_1206 -> Resistors_SMD:R_0805
- R9: renamed from R2; footprint Resistors_SMD:R_1206 -> Resistors_SMD:R_0805
- renumbered C5 to C1, C16 to C3, C2 to C5, C15 to C6, D2 to D1, D6 to D5, RFM69HW1 to RF1
Connections:
- net labels added: BOOT0, BOOT1, OSCIN, OSCOUT, RESET, RTCIN, RTCOUT, STAT_LED, SWDCLK, SWDIO, USB_D+, USB_D-
- net labels removed: LED
- wire segments 129 -> 186
- no-connect marks 1 -> 16
Other:
- moved on the sheet: BARO1, C1, C16, C2, C3, C4, C5, C6, C7, D1, D5, F1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
