File: hardware/console.sch (KiCad schematic (older format))
At the start: 22 parts, among them J2 Micro USB, J3 IGC, Y1 12M

Commit message: Unfinished pcb layouts
Parts:
- removed F1: 1A, Fuse_Holders_and_Fuses:Fuse_SMD1206_Reflow, symbol Polyfuse_Small
- C13, C14: footprint Capacitors_ThroughHole:C_Disc_D5.0mm_W2.5mm_P5.00mm -> Capacitors_SMD:C_0603_HandSoldering
Connections:
- wire segments 95 -> 94
Changed lines of the file:
@@
 F 0 "C14" H 7560 2120 50  0000 L CNN
 F 1 "22pF" H 7560 1970 50  0000 L CNN
-F 2 "Capacitors_ThroughHole:C_Disc_D5.0mm_W2.5mm_P5.00mm" H 7550 2050 50  0001 C CNN
+F 2 "Capacitors_SMD:C_0603_HandSoldering" H 7550 2050 50  0001 C CNN
 F 3 "" H 7550 2050 50  0001 C CNN
 	1    7550 2050
@@
 F 0 "C13" H 7560 1820 50  0000 L CNN
 F 1 "22pF" H 7560 1670 50  0000 L CNN
-F 2 "Capacitors_ThroughHole:C_Disc_D5.0mm_W2.5mm_P5.00mm" H 7550 1750 50  0001 C CNN
+F 2 "Capacitors_SMD:C_0603_HandSoldering" H 7550 1750 50  0001 C CNN
 F 3 "" H 7550 1750 50  0001 C CNN
 	1    7550 1750
@@
 Text GLabel 8300 1250 1    60   Input ~ 0
 3.3V
-Text GLabel 9700 2900 2    60   Input ~ 0
+Text GLabel 9500 2900 2    60   Input ~ 0
 5V
 $Comp
@@
 	9400 3100 9400 3950
 Wire Wire Line
-	9150 2900 9400 2900
+	9150 2900 9500 2900
 $Comp
 L C_Small C17
@@
 Wire Wire Line
 	7900 1350 7900 1400
-$Comp
-L Polyfuse_Small F1
-U 1 1 5A06547F
-P 9500 2900
-F 0 "F1" V 9425 2900 50  0000 C CNN
-F 1 "1A" V 9575 2900 50  0000 C CNN
-F 2 "Fuse_Holders_and_Fuses:Fuse_SMD1206_Reflow" H 9550 2700 50  0001 L CNN
-F 3 "" H 9500 2900 50  0001 C CNN
-	1    9500 2900
-	0    1    1    0
-$EndComp
-Wire Wire Line
-	9600 2900 9700 2900
 Text Label 2400 2850 0    40   ~ 0
 MAX232_TX

Commit message: Unverified attempt on standalone STM32 chip
Parts:
- added R17, R18: 20, Resistors_SMD:R_0805, symbol R_Small
- added R19: 1.5K, Resistors_SMD:R_0805, symbol R_Small
- C19: renamed from C6; footprint Capacitors_SMD:C_1206 -> Capacitors_SMD:C_0805
- C20: renamed from C7; footprint Capacitors_SMD:C_1206 -> Capacitors_SMD:C_0805
- C21: renamed from C8; footprint Capacitors_SMD:C_1206 -> Capacitors_SMD:C_0805
- C22: renamed from C9; footprint Capacitors_SMD:C_1206 -> Capacitors_SMD:C_0805
- C23: renamed from C10; footprint Capacitors_SMD:C_1206 -> Capacitors_SMD:C_0805
- C24: renamed from C17; footprint Capacitors_SMD:C_1206 -> Capacitors_SMD:C_0805
- J5: renamed from J2; footprint Connectors_Molex:USB_Micro-B_Molex_47346-0001 -> OGN Tracker:USB_Micro
- R14: renamed from R4; footprint Resistors_SMD:R_1206 -> Resistors_SMD:R_0805
- R15: renamed from R5; footprint Resistors_SMD:R_1206 -> Resistors_SMD:R_0805
- R16: renamed from R6; footprint Resistors_SMD:R_1206 -> Resistors_SMD:R_0805
- renumbered BLUETOOTH1 to BT1, C13 to C25, C14 to C26, C18 to C27, D3 to D6, D4 to D7, D5 to D8, J3 to J4, MAX232 to MAX1, Y1 to Y3
Connections:
- net labels added: CON_USB_D+, CON_USB_D-
- wire segments 94 -> 101
- no-connect marks 12 -> 11

Commit message: All the used footprints moved to project directory
Parts:
- BT1: footprint OGN Tracker:JDY-08 -> KDR Tracker:JDY-08
- J4: footprint OGN Tracker:RJ45_SOCKET_SHLD -> KDR Tracker:RJ45_SOCKET_SHLD
- J5: footprint OGN Tracker:USB_Micro -> KDR Tracker:USB_Micro
Changed lines of the file:
@@
 F 0 "J4" H 5950 2100 50  0000 C CNN
 F 1 "IGC" H 5600 2100 50  0000 C CNN
-F 2 "OGN Tracker:RJ45_SOCKET_SHLD" H 5750 1600 50  0001 C CNN
+F 2 "KDR Tracker:RJ45_SOCKET_SHLD" H 5750 1600 50  0001 C CNN
 F 3 "" H 5750 1600 50  0001 C CNN
 	1    5750 1600
@@
 F 0 "BT1" H 3150 7150 60  0000 C CNN
 F 1 "JDY-08" H 3700 6250 60  0000 C CNN
-F 2 "OGN Tracker:JDY-08" H 3900 5850 60  0001 C CNN
+F 2 "KDR Tracker:JDY-08" H 3900 5850 60  0001 C CNN
 F 3 "" H 3900 5850 60  0001 C CNN
 	1    3700 6300
@@
 F 0 "J5" H 8650 3550 50  0000 L CNN
 F 1 "Micro USB" H 8650 3450 50  0000 L CNN
-F 2 "OGN Tracker:USB_Micro" H 9000 3050 50  0001 C CNN
+F 2 "KDR Tracker:USB_Micro" H 9000 3050 50  0001 C CNN
 F 3 "" H 9000 3050 50  0001 C CNN
 	1    8850 3100

Commit message: v0.6 routed
Parts:
- removed BT1: JDY-08, KDR Tracker:JDY-08, symbol JDY-08
- removed C24: 100nF, Capacitors_SMD:C_0805, symbol C_Small
- removed R19: 1.5K, Resistors_SMD:R_0805, symbol R_Small
- added BT1: HC-05, KDR Tracker:HC-05, symbol HC-05
- added C12: 1uF, Capacitors_SMD:C_1206, symbol C_Small
- added J6: BT_KEY, Pin_Headers:Pin_Header_Straight_2x01_Pitch2.54mm, symbol CONN_01X02
- added J7: UART, Pin_Headers:Pin_Header_Straight_1x04_Pitch2.54mm, symbol CONN_01X04
- added LED4: LED_BT_STATUS, LEDs:LED_0603, symbol LED_Small
- C25, C26: footprint Capacitors_SMD:C_0603_HandSoldering -> Capacitors_SMD:C_0603
- R17: value 20 -> 100K
- R18: value 20 -> 520
Connections:
- net labels added: BT_KEY, BT_PAIRED
- net labels removed: BT_TX, USB_D+, USB_D-
- wire segments 101 -> 115

Commit message: Components renamed to be more uniform
Parts:
- renumbered BT1 to RF2, MAX1 to U2, CH340G1 to U3, Y3 to Y1
Changed lines of the file:
@@
 $EndDescr
 $Comp
-L MAX232 MAX1
+L MAX232 U2
 U 1 1 59FF8DDB
 P 3700 2350
-F 0 "MAX1" H 3400 3450 50  0000 R CNN
+F 0 "U2" H 3400 3450 60  0000 R CNN
 F 1 "MAX3232" H 3850 2550 50  0000 R CNN
 F 2 "Housings_SOIC:SOIC-16_3.9x9.9mm_Pitch1.27mm" H 3750 1300 50  0001 L CNN
@@
 3.3V
 $Comp
-L Earth #PWR028
+L Earth #PWR29
 U 1 1 59FF8DE3
 P 3700 3550
-F 0 "#PWR028" H 3700 3300 50  0001 C CNN
+F 0 "#PWR29" H 3700 3300 50  0001 C CNN
 F 1 "Earth" H 3700 3400 50  0001 C CNN
 F 2 "" H 3700 3550 50  0001 C CNN
@@
 $EndComp
 $Comp
-L Earth #PWR029
+L Earth #PWR32
 U 1 1 59FF8E0E
 P 5050 2300
-F 0 "#PWR029" H 5050 2050 50  0001 C CNN
+F 0 "#PWR32" H 5050 2050 50  0001 C CNN
 F 1 "Earth" H 5050 2150 50  0001 C CNN
 F 2 "" H 5050 2300 50  0001 C CNN
@@
 $EndComp
 $Comp
-L Earth #PWR030
+L Earth #PWR38
 U 1 1 59FF8E2D
 P 6300 1250
-F 0 "#PWR030" H 6300 1000 50  0001 C CNN
+F 0 "#PWR38" H 6300 1000 50  0001 C CNN
 F 1 "Earth" H 6300 1100 50  0001 C CNN
 F 2 "" H 6300 1250 50  0001 C CNN
@@
 $EndComp
 $Comp
-L Earth #PWR031
+L Earth #PWR34
 U 1 1 59FF8E33
 P 5400 2150
-F 0 "#PWR031" H 5400 1900 50  0001 C CNN
+F 0 "#PWR34" H 5400 1900 50  0001 C CNN
 F 1 "Earth" H 5400 2000 50  0001 C CNN
 F 2 "" H 5400 2150 50  0001 C CNN
@@
 $EndComp
 $Comp
-L +12V #PWR032
+L +12V #PWR37
 U 1 1 59FF8E3C
 P 6100 2150
-F 0 "#PWR032" H 6100 2000 50  0001 C CNN
+F 0 "#PWR37" H 6100 2000 50  0001 C CNN
 F 1 "+12V" H 6100 2290 50  0000 C CNN
 F 2 "" H 6100 2150 50  0001 C CNN
@@
 $EndComp
 $Comp
-L Earth #PWR033
+L Earth #PWR35
 U 1 1 59FF8E4B
 P 5800 2150
-F 0 "#PWR033" H 5800 1900 50  0001 C CNN
+F 0 "#PWR35" H 5800 1900 50  0001 C CNN
 F 1 "Earth" H 5800 2000 50  0001 C CNN
 F 2 "" H 5800 2150 50  0001 C CNN
@@
 $EndComp
 $Comp
-L Earth #PWR034
+L Earth #PWR30
 U 1 1 59FF8E78
 P 4100 1050
-F 0 "#PWR034" H 4100 800 50  0001 C CNN
+F 0 "#PWR30" H 4100 800 50  0001 C CNN
 F 1 "Earth" H 4100 900 50  0001 C CNN
 F 2 "" H 4100 1050 50  0001 C CNN
@@
 CON_OUTPUT
 $Comp
-L CH340G CH340G1
+L CH340G U3
 U 1 1 59FFA19D
 P 9000 1800
-F 0 "CH340G1" H 8850 2500 60  0000 C CNN
+F 0 "U3" H 8850 2500 60  0000 C CNN
 F 1 "CH340G" V 9050 1800 60  0000 C CNN
 F 2 "Housings_SOIC:SOIC-16_3.9x9.9mm_Pitch1.27mm" H 9000 1800 60  0001 C CNN
@@
 $EndComp
 $Comp
-L Crystal Y3
+L Crystal Y1
 U 1 1 59FFA406
 P 8000 1900
-F 0 "Y3" H 8000 2050 50  0000 C CNN
+F 0 "Y1" H 8000 2050 50  0000 C CNN
 F 1 "12M" H 8000 1750 50  0000 C CNN
 F 2 "Crystals:Crystal_HC49-4H_Vertical" H 8000 1900 50  0001 C CNN
@@
 $EndComp
 $Comp
-L Earth #PWR035
+L Earth #PWR39
 U 1 1 59FFEECD
 P 7300 1950
-F 0 "#PWR035" H 7300 1700 50  0001 C CNN
+F 0 "#PWR39" H 7300 1700 50  0001 C CNN
 F 1 "Earth" H 7300 1800 50  0001 C CNN
 F 2 "" H 7300 1950 50  0001 C CNN
@@
 $EndComp
 $Comp
-L Earth #PWR036
+L Earth #PWR41
 U 1 1 59FFF2A6
 P 8400 1650
-F 0 "#PWR036" H 8400 1400 50  0001 C CNN
+F 0 "#PWR41" H 8400 1400 50  0001 C CNN
 F 1 "Earth" H 8400 1500 50  0001 C CNN
 F 2 "" H 8400 1650 50  0001 C CNN
@@
 5V
 $Comp
-L Earth #PWR037
+L Earth #PWR42
 U 1 1 59FFFCBC
 P 8850 3600
-F 0 "#PWR037" H 8850 3350 50  0001 C CNN
+F 0 "#PWR42" H 8850 3350 50  0001 C CNN
 F 1 "Earth" H 8850 3450 50  0001 C CNN
 F 2 "" H 8850 3600 50  0001 C CNN
@@
 $EndComp
 $Comp
-L Earth #PWR038
+L Earth #PWR40
 U 1 1 5A06460D
 P 7900 1400
-F 0 "#PWR038" H 7900 1150 50  0001 C CNN
+F 0 "#PWR40" H 7900 1150 50  0001 C CNN
 F 1 "Earth" H 7900 1250 50  0001 C CNN
 F 2 "" H 7900 1400 50  0001 C CNN
@@
 $EndComp
 $Comp
-L Earth #PWR039
+L Earth #PWR43
 U 1 1 5A2F3AFB
 P 9300 5200
-F 0 "#PWR039" H 9300 4950 50  0001 C CNN
+F 0 "#PWR43" H 9300 4950 50  0001 C CNN
 F 1 "Earth" H 9300 5050 50  0001 C CNN
 F 2 "" H 9300 5200 50  0001 C CNN
@@
 CON_TX
 $Comp
-L HC-05 BT1
+L HC-05 RF2
 U 1 1 5A2F470E
 P 4350 6250
-F 0 "BT1" H 3750 7100 60  0000 L CNN
+F 0 "RF2" H 3750 7100 60  0000 L CNN
 F 1 "HC-05" H 3750 7000 60  0000 L CNN
 F 2 "KDR Tracker:HC-05" H 3450 7100 60  0001 C CNN
@@
 $EndComp
 $Comp
-L Earth #PWR040
+L Earth #PWR28
 U 1 1 5A2F528C
 P 3350 7200
-F 0 "#PWR040" H 3350 6950 50  0001 C CNN
+F 0 "#PWR28" H 3350 6950 50  0001 C CNN
 F 1 "Earth" H 3350 7050 50  0001 C CNN
 F 2 "" H 3350 7200 50  0001 C CNN
@@
 $EndComp
 $Comp
-L Earth #PWR041
+L Earth #PWR31
 U 1 1 5A2F52EE
 P 4700 7450
-F 0 "#PWR041" H 4700 7200 50  0001 C CNN
+F 0 "#PWR31" H 4700 7200 50  0001 C CNN
 F 1 "Earth" H 4700 7300 50  0001 C CNN
 F 2 "" H 4700 7450 50  0001 C CNN
@@
 $EndComp
 $Comp
-L Earth #PWR042
+L Earth #PWR33
 U 1 1 5A2F5336
 P 5350 6950
-F 0 "#PWR042" H 5350 6700 50  0001 C CNN
+F 0 "#PWR33" H 5350 6700 50  0001 C CNN
 F 1 "Earth" H 5350 6800 50  0001 C CNN
 F 2 "" H 5350 6950 50  0001 C CNN
@@
 Connection ~ 5500 5400
 $Comp
-L Earth #PWR043
+L Earth #PWR36
 U 1 1 5A2F7F1D
 P 5850 5500
-F 0 "#PWR043" H 5850 5250 50  0001 C CNN
+F 0 "#PWR36" H 5850 5250 50  0001 C CNN
 F 1 "Earth" H 5850 5350 50  0001 C CNN
 F 2 "" H 5850 5500 50  0001 C CNN

Commit message: Naming library properly
Parts:
- J4: footprint KDR Tracker:RJ45_SOCKET_SHLD -> Ked Tracker:RJ45_SOCKET_SHLD
- J5: footprint KDR Tracker:USB_Micro -> Ked Tracker:USB_Micro
- RF2: footprint KDR Tracker:HC-05 -> Ked Tracker:HC-05
Changed lines of the file:
@@
 LIBS:valves
 LIBS:stm32
-LIBS:ogntracker
+LIBS:kedtracker
 LIBS:switches
 LIBS:kedder
-LIBS:ogntracker-cache
+LIBS:kedtracker-cache
 EELAYER 25 0
 EELAYER END
@@
 F 0 "J4" H 5950 2100 50  0000 C CNN
 F 1 "IGC" H 5600 2100 50  0000 C CNN
-F 2 "KDR Tracker:RJ45_SOCKET_SHLD" H 5750 1600 50  0001 C CNN
+F 2 "Ked Tracker:RJ45_SOCKET_SHLD" H 5750 1600 50  0001 C CNN
 F 3 "" H 5750 1600 50  0001 C CNN
 	1    5750 1600
@@
 F 0 "J5" H 8650 3550 50  0000 L CNN
 F 1 "Micro USB" H 8650 3450 50  0000 L CNN
-F 2 "KDR Tracker:USB_Micro" H 9000 3050 50  0001 C CNN
+F 2 "Ked Tracker:USB_Micro" H 9000 3050 50  0001 C CNN
 F 3 "" H 9000 3050 50  0001 C CNN
 	1    8850 3100
@@
 F 0 "RF2" H 3750 7100 60  0000 L CNN
 F 1 "HC-05" H 3750 7000 60  0000 L CNN
-F 2 "KDR Tracker:HC-05" H 3450 7100 60  0001 C CNN
+F 2 "Ked Tracker:HC-05" H 3450 7100 60  0001 C CNN
 F 3 "" H 3450 7100 60  0000 C CNN
 	1    4350 6250
