File: hardware/console.sch (KiCad schematic (older format))
At the start: 26 parts, among them J4 IGC, J5 Micro USB, J6 BT_KEY, J7 UART, U2 MAX3232, U3 CH340G, Y1 12M

Commit message: Update schematics to latest KiCAD version
Parts:
- C12, C19, C20, C21, C22, C23, C25, C26, C27: symbol C_Small -> kedtracker-rescue:C_Small
- D6, D7, D8: symbol D_Small -> kedtracker-rescue:D_Small
- J4: symbol RJ45 -> kedtracker-rescue:RJ45
- J5: symbol USB_OTG -> kedtracker-rescue:USB_OTG
- J6: symbol CONN_01X02 -> kedtracker-rescue:CONN_01X02
- J7: symbol CONN_01X04 -> kedtracker-rescue:CONN_01X04
- LED4: symbol LED_Small -> kedtracker-rescue:LED_Small
- R14, R15, R16, R17, R18: symbol R_Small -> kedtracker-rescue:R_Small
- RF2: symbol HC-05 -> kedtracker-rescue:HC-05
- U2: symbol MAX232 -> kedtracker-rescue:MAX232
- U3: symbol CH340G -> kedtracker-rescue:CH340G
- Y1: symbol Crystal -> kedtracker-rescue:Crystal
Changed lines of the file:
@@
-EESchema Schematic File Version 2
-LIBS:power
-LIBS:device
-LIBS:transistors
-LIBS:conn
-LIBS:linear
-LIBS:regul
-LIBS:74xx
-LIBS:cmos4000
-LIBS:adc-dac
-LIBS:memory
-LIBS:xilinx
-LIBS:microcontrollers
-LIBS:dsp
-LIBS:microchip
-LIBS:analog_switches
-LIBS:motorola
-LIBS:texas
-LIBS:intel
-LIBS:audio
-LIBS:interface
-LIBS:digital-audio
-LIBS:philips
-LIBS:display
-LIBS:cypress
-LIBS:siliconi
-LIBS:opto
-LIBS:atmel
-LIBS:contrib
-LIBS:valves
-LIBS:stm32
-LIBS:kedtracker
-LIBS:switches
-LIBS:kedder
+EESchema Schematic File Version 4
 LIBS:kedtracker-cache
-EELAYER 25 0
+EELAYER 26 0
 EELAYER END
 $Descr A4 11693 8268
@@
 $EndDescr
 $Comp
-L MAX232 U2
+L kedtracker-rescue:MAX232 U2
 U 1 1 59FF8DDB
 P 3700 2350
@@
 3.3V
 $Comp
-L Earth #PWR030
+L kedtracker-rescue:Earth #PWR030
 U 1 1 59FF8DE3
 P 3700 3550
@@
 $EndComp
 $Comp
-L C_Small C21
+L kedtracker-rescue:C_Small C21
 U 1 1 59FF8DE9
 P 4600 1600
@@
 $EndComp
 $Comp
-L C_Small C19
+L kedtracker-rescue:C_Small C19
 U 1 1 59FF8DF4
 P 2650 1600
@@
 $EndComp
 $Comp
-L C_Small C22
+L kedtracker-rescue:C_Small C22
 U 1 1 59FF8DFF
 P 4750 1950
@@
 $EndComp
 $Comp
-L C_Small C23
+L kedtracker-rescue:C_Small C23
 U 1 1 59FF8E06
 P 4750 2250
@@
 $EndComp
 $Comp
-L Earth #PWR031
+L kedtracker-rescue:Earth #PWR031
 U 1 1 59FF8E0E
 P 5050 2300
@@
 $EndComp
 $Comp
-L RJ45 J4
+L kedtracker-rescue:RJ45 J4
 U 1 1 59FF8E19
 P 5750 1600
@@
 $EndComp
 $Comp
-L Earth #PWR032
+L kedtracker-rescue:Earth #PWR032
 U 1 1 59FF8E2D
 P 6300 1250
@@
 $EndComp
 $Comp
-L Earth #PWR033
+L kedtracker-rescue:Earth #PWR033
 U 1 1 59FF8E33
 P 5400 2150
@@
 $EndComp
 $Comp
-L +12V #PWR034
+L kedtracker-rescue:+12V #PWR034
 U 1 1 59FF8E3C
 P 6100 2150
@@
 $EndComp
 $Comp
-L Earth #PWR035
+L kedtracker-rescue:Earth #PWR035
 U 1 1 59FF8E4B
 P 5800 2150
@@
 3.3V
 $Comp
-L C_Small C20
+L kedtracker-rescue:C_Small C20
 U 1 1 59FF8E6F
 P 3900 1050
@@
 $EndComp
 $Comp
-L Earth #PWR036
+L kedtracker-rescue:Earth #PWR036
 U 1 1 59FF8E78
 P 4100 1050
@@
 $EndComp
 $Comp
-L D_Small D6
+L kedtracker-rescue:D_Small D6
 U 1 1 59FF8EA1
 P 2200 2850
@@
 $EndComp
 $Comp
-L R_Small R14
+L kedtracker-rescue:R_Small R14
 U 1 1 59FF8EA9
 P 2200 2650
@@
 CON_OUTPUT
 $Comp
-L CH340G U3
+L kedtracker-rescue:CH340G U3
 U 1 1 59FFA19D
 P 9000 1800
@@
 $EndComp
 $Comp
-L USB_OTG J5
+L kedtracker-rescue:USB_OTG J5
 U 1 1 59FFA20C
 P 8850 3100
@@
 $EndComp
 $Comp
-L Crystal Y1
+L kedtracker-rescue:Crystal Y1
 U 1 1 59FFA406
 P 8000 1900
@@
 CON_TX
 $Comp
-L D_Small D8
+L kedtracker-rescue:D_Small D8
 U 1 1 59FFDDAC
 P 10050 1350
@@
 $EndComp
 $Comp
-L R_Small R16
+L kedtracker-rescue:R_Small R16
 U 1 1 59FFE1F4
 P 10050 1150
@@
 $EndComp
 $Comp
-L C_Small C26
+L kedtracker-rescue:C_Small C26
 U 1 1 59FFEA83
 P 7550 2050
@@
 $EndComp
 $Comp
-L C_Small C25
+L kedtracker-rescue:C_Small C25
 U 1 1 59FFEAE2
 P 7550 1750
@@
 $EndComp
 $Comp
-L Earth #PWR037
+L kedtracker-rescue:Earth #PWR037
 U 1 1 59FFEECD
 P 7300 1950
@@
 $EndComp
 $Comp
-L Earth #PWR038
+L kedtracker-rescue:Earth #PWR038
 U 1 1 59FFF2A6
 P 8400 1650
@@
 5V
 $Comp
-L Earth #PWR039
+L kedtracker-rescue:Earth #PWR039
 U 1 1 59FFFCBC
 P 8850 3600
@@
 	8000 3950 8000 2250
 $Comp
-L C_Small C27
+L kedtracker-rescue:C_Small C27
 U 1 1 5A0644CA
 P 8050 1350
@@
 $EndComp
 $Comp
-L Earth #PWR040
+L kedtracker-rescue:Earth #PWR040
 U 1 1 5A06460D
 P 7900 1400
@@
 	9200 3300 9200 3550
 $Comp
-L CONN_01X04 J7
+L kedtracker-rescue:CONN_01X04 J7
 U 1 1 5A2F37E8
 P 9600 4950
@@
 $EndComp
 $Comp
-L Earth #PWR041
+L kedtracker-rescue:Earth #PWR041
 U 1 1 5A2F3AFB
 P 9300 5200
@@
 CON_TX
 $Comp
-L HC-05 RF2
+L kedtracker-rescue:HC-05 RF2
 U 1 1 5A2F470E
 P 4350 6250
@@
 $EndComp
 $Comp
-L Earth #PWR042
+L kedtracker-rescue:Earth #PWR042
 U 1 1 5A2F528C
 P 3350 7200
@@
 $EndComp
 $Comp
-L Earth #PWR043
+L kedtracker-rescue:Earth #PWR043
 U 1 1 5A2F52EE
 P 4700 7450
@@
 $EndComp
 $Comp
-L Earth #PWR044
+L kedtracker-rescue:Earth #PWR044
 U 1 1 5A2F5336
 P 5350 6950
@@
 	3100 5650 3450 5650
 $Comp
-L D_Small D7
+L kedtracker-rescue:D_Small D7
 U 1 1 5A2F5939
 P 3000 5650
@@
 $EndComp
 $Comp
-L R_Small R15
+L kedtracker-rescue:R_Small R15
 U 1 1 5A2F593F
 P 3000 5400
@@
 CON_TX
 $Comp
-L C_Small C12
+L kedtracker-rescue:C_Small C12
 U 1 1 5A2F679C
 P 3150 6950
@@
 	5500 5650 5250 5650
 $Comp
-L CONN_01X02 J6
+L kedtracker-rescue:CONN_01X02 J6
 U 1 1 5A2F782C
 P 5300 5200
@@
 	5500 5250 5500 5650
 $Comp
-L R_Small R17
+L kedtracker-rescue:R_Small R17
 U 1 1 5A2F7D4B
 P 5650 5400
@@
 Connection ~ 5500 5400
 $Comp
-L Earth #PWR045
+L kedtracker-rescue:Earth #PWR045
 U 1 1 5A2F7F1D
 P 5850 5500
@@
 BT_KEY
 $Comp
-L LED_Small LED4
+L kedtracker-rescue:LED_Small LED4
 U 1 1 5A2F840B
 P 6150 6250
@@
 $EndComp
 $Comp
-L R_Small R18
+L kedtracker-rescue:R_Small R18
 U 1 1 5A2F84BF
 P 5850 6250
@@
 	9150 3100 9400 3100
 $Comp
-L Earth #PWR046
+L kedtracker-rescue:Earth #PWR046
 U 1 1 5A7708E8
 P 6350 6350
