File: hardware/kedtracker.kicad_pcb (KiCad board)
At the start: 2 copper layers, 82.7 x 56.6 mm, 80 parts, among them J1 ANT, J2 SWD, J3 BOOT, J4 IGC, J5 Micro USB, J6 BT_KEY, J7 UART, J8 VK2828U7G5LF, J9 Micro SD Reader, SW1 RESET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

Commit message: Naming library properly
Parts:
- B1: footprint KDR Tracker:Buck_Converter_Sm -> Ked Tracker:Buck_Converter_Sm
- B2: footprint KDR Tracker:BMP280 -> Ked Tracker:BMP280
- J1: footprint KDR Tracker:SMA_CONN -> Ked Tracker:SMA_CONN
- J4: footprint KDR Tracker:RJ45_SOCKET_SHLD -> Ked Tracker:RJ45_SOCKET_SHLD
- J5: footprint KDR Tracker:USB_Micro -> Ked Tracker:USB_Micro
- J8: footprint KDR Tracker:Molex_PicoBlade_53047-0610_06x1.25mm_Straight -> Ked Tracker:Molex_PicoBlade_53047-0610_06x1.25mm_Straight
- J9: footprint KDR Tracker:SDCARD_BOMB -> Ked Tracker:SDCARD_BOMB
- RF1: footprint KDR Tracker:RFM69HW -> Ked Tracker:RFM69HW
- RF2: footprint KDR Tracker:HC-05 -> Ked Tracker:HC-05
Other:
- board text added: "Ked Tracker v0.6"
- board text added: "Ked Tracker v0.6 2017"
- board text added: "Open Glider Network Tracker For Hammond-1593L enclosure Based on design by http://glidernet.org For more info visit https://github.com/kedder/kedtracker"
- board text removed: "KDR Tracker v0.6"
- board text removed: "KDR Tracker v0.6 2017"
- board text removed: "Open Glider Network Tracker For Hammond-1593L enclosure Based on design by http://glidernet.org For more info visit https://github.com/kedder/kdrtracker"
Changed lines of the file:
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@@
   (page A4)
   (title_block
-    (title "KDR Tracker")
+    (title "Ked Tracker")
     (date 2017-12-16)
     (rev 0.6)
@@
     (pad 1 np_thru_hole circle (at 0 0) (size 3.2 3.2) (drill 3.2) (layers *.Cu *.Mask))
   )
-  (module "KDR Tracker:HC-05" (layer F.Cu)
+  (module "Ked Tracker:HC-05" (layer F.Cu)
     (at 126.128 91.872 90)
     (fp_text reference RF2 (at 5.6 -23.2 90) (layer F.SilkS)
@@
       (net 33 /5V_PROT))
   )
-  (module "KDR Tracker:USB_Micro" (layer F.Cu)
+  (module "Ked Tracker:USB_Micro" (layer F.Cu)
     (at 179.93 56.75 180)
     (descr http://www.molex.com/pdm_docs/sd/473460001_sd.pdf)
@@
     )
   )
-  (module "KDR Tracker:SDCARD_BOMB" (layer F.Cu)
+  (module "Ked Tracker:SDCARD_BOMB" (layer F.Cu)
     (at 101.28 70.028 270)
     (fp_text reference J9 (at 0 -4.5 270) (layer F.SilkS)
@@
     )
   )
-  (module "KDR Tracker:SMA_CONN" (layer F.Cu)
+  (module "Ked Tracker:SMA_CONN" (layer F.Cu)
     (at 178.232 92.888 270)
     (tags "SMA Connector")
@@
     )
   )
-  (module "KDR Tracker:Molex_PicoBlade_53047-0610_06x1.25mm_Straight" (layer F.Cu)
+  (module "Ked Tracker:Molex_PicoBlade_53047-0610_06x1.25mm_Straight" (layer F.Cu)
     (at 160.274 54.71 270)
     (descr "Molex PicoBlade, single row, top entry type, through hole, PN:53047-0610")
@@
     )
   )
-  (module "KDR Tracker:BMP280" (layer F.Cu)
+  (module "Ked Tracker:BMP280" (layer F.Cu)
     (at 129.54 47.625 180)
     (fp_text reference B2 (at 0 -5.08 180) (layer F.SilkS)
@@
       (net 1 3.3V))
   )
-  (module "KDR Tracker:Buck_Converter_Sm" (layer F.Cu)
+  (module "Ked Tracker:Buck_Converter_Sm" (layer F.Cu)
     (at 171.628 59.36 90)
     (fp_text reference B1 (at -2.54 0 180) (layer F.SilkS)
@@
       (net 2 5V))
   )
-  (module "KDR Tracker:RFM69HW" (layer F.Cu)
+  (module "Ked Tracker:RFM69HW" (layer F.Cu)
     (at 147.066 86.36)
     (fp_text reference RF1 (at 0 0) (layer F.SilkS)
@@
       (net 7 Earth))
   )
-  (module "KDR Tracker:RJ45_SOCKET_SHLD" (layer F.Cu)
+  (module "Ked Tracker:RJ45_SOCKET_SHLD" (layer F.Cu)
     (at 178.105 73.965 90)
     (tags RJ45)
@@
     (effects (font (size 1.5 1.5) (thickness 0.3)) (justify mirror))
   )
-  (gr_text "KDR Tracker\nv0.6\n2017" (at 172.72 92.71) (layer F.SilkS)
+  (gr_text "Ked Tracker\nv0.6\n2017" (at 172.72 92.71) (layer F.SilkS)
     (effects (font (size 1.5 1.5) (thickness 0.3)) (justify right))
   )
-  (gr_text "Open Glider Network Tracker\n\nFor Hammond-1593L enclosure\n\nBased on design by http://glidernet.org\nFor more info visit\nhttps://github.com/kedder/kdrtracker" (at 133.096 98.044 270) (layer B.SilkS)
+  (gr_text "Open Glider Network Tracker\n\nFor Hammond-1593L enclosure\n\nBased on design by http://glidernet.org\nFor more info visit\nhttps://github.com/kedder/kedtracker" (at 133.096 98.044 270) (layer B.SilkS)
     (effects (font (size 1 1) (thickness 0.15)) (justify left mirror))
   )
-  (gr_text "KDR Tracker v0.6" (at 141.224 98.044 270) (layer B.SilkS)
+  (gr_text "Ked Tracker v0.6" (at 141.224 98.044 270) (layer B.SilkS)
     (effects (font (size 2.5 2.5) (thickness 0.4)) (justify left mirror))
   )
