File: hardware/kedtracker.sch (KiCad schematic (older format))
At the start: 50 parts, among them J1 ANT, J2 SWD, J3 BOOT, J8 VK2828U7G5LF, J9 Micro SD Reader, SW1 RESET, U1 LM2936-3.3, Y2 8MHz

Commit message: Naming library properly
Parts:
- B1: footprint KDR Tracker:Buck_Converter_Sm -> Ked Tracker:Buck_Converter_Sm
- B2: footprint KDR Tracker:BMP280 -> Ked Tracker:BMP280
- J1: footprint KDR Tracker:SMA_CONN -> Ked Tracker:SMA_CONN
- J8: footprint KDR Tracker:Molex_PicoBlade_53047-0610_06x1.25mm_Straight -> Ked Tracker:Molex_PicoBlade_53047-0610_06x1.25mm_Straight
- J9: footprint KDR Tracker:SDCARD_BOMB -> Ked Tracker:SDCARD_BOMB
- RF1: footprint KDR Tracker:RFM69HW -> Ked Tracker:RFM69HW
Changed lines of the file:
@@
 LIBS:valves
 LIBS:stm32
-LIBS:ogntracker
+LIBS:kedtracker
 LIBS:switches
 LIBS:kedder
-LIBS:ogntracker-cache
+LIBS:kedtracker-cache
 EELAYER 25 0
 EELAYER END
@@
 F 0 "RF1" H 2800 5600 60  0000 L CNN
 F 1 "RFM69HW" H 2700 4500 60  0000 C CNN
-F 2 "KDR Tracker:RFM69HW" H 2700 4950 60  0001 C CNN
+F 2 "Ked Tracker:RFM69HW" H 2700 4950 60  0001 C CNN
 F 3 "" H 2700 4950 60  0001 C CNN
 	1    2700 4950
@@
 F 0 "J8" H 1400 3000 60  0000 L CNN
 F 1 "VK2828U7G5LF" H 1800 3250 40  0000 C CNN
-F 2 "KDR Tracker:Molex_PicoBlade_53047-0610_06x1.25mm_Straight" H 2250 3700 40  0001 C CNN
+F 2 "Ked Tracker:Molex_PicoBlade_53047-0610_06x1.25mm_Straight" H 2250 3700 40  0001 C CNN
 F 3 "" H 2250 3700 40  0001 C CNN
 	1    1800 3500
@@
 F 0 "J1" H 1810 5670 50  0000 C CNN
 F 1 "ANT" V 1915 5550 50  0000 C CNN
-F 2 "KDR Tracker:SMA_CONN" H 1800 5550 50  0001 C CNN
+F 2 "Ked Tracker:SMA_CONN" H 1800 5550 50  0001 C CNN
 F 3 "" H 1800 5550 50  0001 C CNN
 	1    1800 5550
@@
 F 0 "B2" H 8850 4400 60  0000 C CNN
 F 1 "BMP280" H 8950 4100 60  0000 C CNN
-F 2 "KDR Tracker:BMP280" H 9000 3750 60  0001 C CNN
+F 2 "Ked Tracker:BMP280" H 9000 3750 60  0001 C CNN
 F 3 "" H 9000 3750 60  0001 C CNN
 	1    8950 3950
@@
 F 0 "B1" H 1750 1700 60  0000 L CNN
 F 1 "BUCK_CVTR" H 2050 1600 40  0000 L CNN
-F 2 "KDR Tracker:Buck_Converter_Sm" H 1800 1450 60  0001 C CNN
+F 2 "Ked Tracker:Buck_Converter_Sm" H 1800 1450 60  0001 C CNN
 F 3 "" H 1800 1450 60  0001 C CNN
 	1    2100 1450
@@
 F 0 "J9" H 5250 7150 50  0000 C CNN
 F 1 "Micro SD Reader" H 6550 7150 50  0000 R CNN
-F 2 "KDR Tracker:SDCARD_BOMB" H 7950 7150 50  0001 C CNN
+F 2 "Ked Tracker:SDCARD_BOMB" H 7950 7150 50  0001 C CNN
 F 3 "" H 5900 6550 50  0001 C CNN
 	1    5900 6450
