File: hardware/kedtracker.sch (KiCad schematic (older format))
At the start: 50 parts, among them J1 ANT, J2 SWD, J3 BOOT, J8 VK2828U7G5LF, J9 Micro SD Reader, SW1 RESET, U1 LM2936-3.3, Y2 8MHz

Commit message: Prepare fabrication layer for assembly
* Proper placement of labels on F.Fab layer
* Element outlines
* Correct values of used components
* LED values indicate color, rather then function
Parts:
- D1: value 1N4001 -> SS14
- F1: value 0.5A -> 0.2A
- J9: value Micro SD Reader -> SDCARD_READER
- LED1: value STATUS_PANEL -> GREEN
- LED2: value STATUS_SMD -> YELLOW
- LED3: value LED_BT -> BLUE
- LED5: value PWR -> RED
- LS1: value Buzzer -> BUZZER
- R1: value 82 -> 100
- R2, R3: value 330 -> 520
- R7: value 82 -> 820
- U1: value LM2936-3.3 -> LM3940
- Y2: value 8MHz -> 8M
Changed lines of the file:
@@
 P 850 1600
 F 0 "D1" H 850 1700 50  0000 C CNN
-F 1 "1N4001" H 850 1500 50  0000 C CNN
+F 1 "SS14" H 850 1500 50  0000 C CNN
 F 2 "Diodes_SMD:D_SMA_Standard" H 850 1600 50  0001 C CNN
 F 3 "" H 850 1600 50  0001 C CNN
@@
 P 5900 6450
 F 0 "J9" H 5250 7150 50  0000 C CNN
-F 1 "Micro SD Reader" H 6550 7150 50  0000 R CNN
+F 1 "SDCARD_READER" H 6550 7150 50  0000 R CNN
 F 2 "Ked Tracker:SDCARD_BOMB" H 7950 7150 50  0001 C CNN
 F 3 "" H 5900 6550 50  0001 C CNN
@@
 P 8050 5550
 F 0 "R7" V 7950 5500 50  0000 L CNN
-F 1 "82" V 8050 5500 40  0000 L CNN
+F 1 "820" V 8050 5500 40  0000 L CNN
 F 2 "Resistors_SMD:R_0805" H 8050 5550 50  0001 C CNN
 F 3 "" H 8050 5550 50  0001 C CNN
@@
 P 7700 5550
 F 0 "LED3" H 7700 5650 50  0000 C CNN
-F 1 "LED_BT" H 7700 5450 50  0000 C CNN
+F 1 "BLUE" H 7700 5450 50  0000 C CNN
 F 2 "LEDs:LED_D5.0mm_Horizontal_O3.81mm_Z3.0mm" H 7700 5550 50  0001 C CNN
 F 3 "" H 7700 5550 50  0001 C CNN
@@
 P 1950 6500
 F 0 "LS1" H 2000 6725 50  0000 R CNN
-F 1 "Buzzer" H 2000 6650 50  0000 R CNN
+F 1 "BUZZER" H 2000 6650 50  0000 R CNN
 F 2 "Buzzers_Beepers:Buzzer_12x9.5RM7.6" H 1950 6300 50  0001 C CNN
 F 3 "" H 1940 6450 50  0001 C CNN
@@
 P 3400 1450
 F 0 "U1" H 3250 1575 50  0000 C CNN
-F 1 "LM2936-3.3" H 3400 1575 50  0000 L CNN
+F 1 "LM3940" H 3400 1575 50  0000 L CNN
 F 2 "TO_SOT_Packages_SMD:SOT-223-3Lead_TabPin2" H 3400 1675 50  0001 C CIN
 F 3 "" H 3400 1400 50  0001 C CNN
@@
 P 850 1100
 F 0 "F1" V 775 1100 50  0000 C CNN
-F 1 "0.5A" V 925 1100 50  0000 C CNN
+F 1 "0.2A" V 925 1100 50  0000 C CNN
 F 2 "Fuse_Holders_and_Fuses:Fuse_SMD1206_Reflow" H 900 900 50  0001 L CNN
 F 3 "" H 850 1100 50  0001 C CNN
@@
 P 8050 1300
 F 0 "Y2" H 8050 1400 50  0000 C CNN
-F 1 "8MHz" H 8050 1200 50  0000 C CNN
+F 1 "8M" H 8050 1200 50  0000 C CNN
 F 2 "Crystals:Crystal_SMD_HC49-SD" H 8050 1300 50  0001 C CNN
 F 3 "" H 8050 1300 50  0001 C CNN
@@
 P 2350 7450
 F 0 "R2" H 2380 7470 50  0000 L CNN
-F 1 "330" H 2380 7410 50  0000 L CNN
+F 1 "520" H 2380 7410 50  0000 L CNN
 F 2 "Resistors_SMD:R_0805" H 2350 7450 50  0001 C CNN
 F 3 "" H 2350 7450 50  0001 C CNN
@@
 P 1850 7450
 F 0 "LED2" H 1800 7575 50  0000 L CNN
-F 1 "STATUS_SMD" H 1675 7350 50  0000 L CNN
+F 1 "YELLOW" H 1700 7350 50  0000 L CNN
 F 2 "LEDs:LED_0603" V 1850 7450 50  0001 C CNN
 F 3 "" V 1850 7450 50  0001 C CNN
@@
 P 1850 7100
 F 0 "LED1" H 1800 7225 50  0000 L CNN
-F 1 "STATUS_PANEL" H 1675 7000 50  0000 L CNN
+F 1 "GREEN" H 1750 7000 50  0000 L CNN
 F 2 "LEDs:LED_D5.0mm_Horizontal_O3.81mm_Z3.0mm" V 1850 7100 50  0001 C CNN
 F 3 "" V 1850 7100 50  0001 C CNN
@@
 P 2350 7100
 F 0 "R1" H 2380 7120 50  0000 L CNN
-F 1 "82" H 2380 7060 50  0000 L CNN
+F 1 "100" H 2380 7060 50  0000 L CNN
 F 2 "Resistors_SMD:R_0805" H 2350 7100 50  0001 C CNN
 F 3 "" H 2350 7100 50  0001 C CNN
@@
 P 4100 1850
 F 0 "LED5" H 4050 1975 50  0000 L CNN
-F 1 "PWR" H 4000 1750 50  0000 L CNN
+F 1 "RED" H 4000 1750 50  0000 L CNN
 F 2 "LEDs:LED_0603" V 4100 1850 50  0001 C CNN
 F 3 "" V 4100 1850 50  0001 C CNN
@@
 P 4100 1600
 F 0 "R3" H 4130 1620 50  0000 L CNN
-F 1 "330" H 4130 1560 50  0000 L CNN
+F 1 "520" H 4130 1560 50  0000 L CNN
 F 2 "Resistors_SMD:R_0805" H 4100 1600 50  0001 C CNN
 F 3 "" H 4100 1600 50  0001 C CNN

Commit message: Changes and fixes for 0.7
* Different 4-pin reset button (because I have a lot of those)
* Bluethooth "paired" and "status" leds swapped - dashboard
  led will show "paired" status and will not annoyingly blink all
  the time
Connections:
- wire segments 171 -> 172
Other:
- moved on the sheet: LED3
Changed lines of the file:
@@
 F 3 "" H 7700 5550 50  0001 C CNN
 	1    7700 5550
-	-1   0    0    1
-$EndComp
-Text GLabel 7400 5550 0    40   Input ~ 0
-3.3V
+	1    0    0    -1
+$EndComp
 $Comp
 L Speaker LS1
@@
 	1    0    0    -1
 $EndComp
+$Comp
+L Earth #PWR?
+U 1 1 5A76FDB7
+P 7400 5650
+F 0 "#PWR?" H 7400 5400 50  0001 C CNN
+F 1 "Earth" H 7400 5500 50  0001 C CNN
+F 2 "" H 7400 5650 50  0001 C CNN
+F 3 "" H 7400 5650 50  0001 C CNN
+	1    7400 5650
+	1    0    0    -1
+$EndComp
+Wire Wire Line
+	7400 5550 7400 5650
 $EndSCHEMATC

Commit message: Updates for power supply and reset button
Parts:
- added D2: SS14, Diodes_SMD:D_SMA_Standard, symbol D_Schottky
- added R19: 10K, Resistors_SMD:R_0805, symbol R_Small
- SW1: footprint Buttons_Switches_SMD:SW_SPST_REED_CT05-XXXX-G1 -> Buttons_Switches_SMD:SW_SPST_SKQG
Connections:
- net labels added: 5V_OUT
- wire segments 172 -> 177
Other:
- moved on the sheet: C3, C6, F2, LED5, R3, U1
Changed lines of the file:
@@
 	1    0    0    -1
 $EndComp
-Text GLabel 2650 1200 1    40   Input ~ 0
+Text GLabel 2500 950  0    40   Input ~ 0
 5V
 $Comp
@@
 L Earth #PWR013
 U 1 1 5A023604
-P 3400 1850
-F 0 "#PWR013" H 3400 1600 50  0001 C CNN
-F 1 "Earth" H 3400 1700 50  0001 C CNN
-F 2 "" H 3400 1850 50  0001 C CNN
-F 3 "" H 3400 1850 50  0001 C CNN
-	1    3400 1850
-	1    0    0    -1
-$EndComp
-Text GLabel 4250 1450 2    40   Input ~ 0
+P 3500 1350
+F 0 "#PWR013" H 3500 1100 50  0001 C CNN
+F 1 "Earth" H 3500 1200 50  0001 C CNN
+F 2 "" H 3500 1350 50  0001 C CNN
+F 3 "" H 3500 1350 50  0001 C CNN
+	1    3500 1350
+	1    0    0    -1
+$EndComp
+Text GLabel 4350 950  2    40   Input ~ 0
 3.3V
 $Comp
 L C_Small C6
 U 1 1 5A02380C
-P 3750 1650
-F 0 "C6" H 3760 1720 50  0000 L CNN
-F 1 "47uF" H 3760 1570 50  0000 L CNN
-F 2 "Capacitors_SMD:C_1210" H 3750 1650 50  0001 C CNN
-F 3 "" H 3750 1650 50  0001 C CNN
-	1    3750 1650
+P 3850 1150
+F 0 "C6" H 3860 1220 50  0000 L CNN
+F 1 "47uF" H 3860 1070 50  0000 L CNN
+F 2 "Capacitors_SMD:C_1210" H 3850 1150 50  0001 C CNN
+F 3 "" H 3850 1150 50  0001 C CNN
+	1    3850 1150
 	1    0    0    -1
 $EndComp
@@
 L Earth #PWR014
 U 1 1 5A023990
-P 3750 1850
-F 0 "#PWR014" H 3750 1600 50  0001 C CNN
-F 1 "Earth" H 3750 1700 50  0001 C CNN
-F 2 "" H 3750 1850 50  0001 C CNN
-F 3 "" H 3750 1850 50  0001 C CNN
-	1    3750 1850
+P 3850 1350
+F 0 "#PWR014" H 3850 1100 50  0001 C CNN
+F 1 "Earth" H 3850 1200 50  0001 C CNN
+F 2 "" H 3850 1350 50  0001 C CNN
+F 3 "" H 3850 1350 50  0001 C CNN
+	1    3850 1350
 	1    0    0    -1
 $EndComp
@@
 L C_Small C3
 U 1 1 5A024206
-P 3000 1650
-F 0 "C3" H 3010 1720 50  0000 L CNN
-F 1 "1uF" H 3010 1570 50  0000 L CNN
-F 2 "Capacitors_SMD:C_1206" H 3000 1650 50  0001 C CNN
-F 3 "" H 3000 1650 50  0001 C CNN
-	1    3000 1650
+P 3100 1150
+F 0 "C3" H 3110 1220 50  0000 L CNN
+F 1 "1uF" H 3110 1070 50  0000 L CNN
+F 2 "Capacitors_SMD:C_1206" H 3100 1150 50  0001 C CNN
+F 3 "" H 3100 1150 50  0001 C CNN
+	1    3100 1150
 	1    0    0    -1
 $EndComp
@@
 L Earth #PWR015
 U 1 1 5A0243BD
-P 3000 1850
-F 0 "#PWR015" H 3000 1600 50  0001 C CNN
-F 1 "Earth" H 3000 1700 50  0001 C CNN
-F 2 "" H 3000 1850 50  0001 C CNN
-F 3 "" H 3000 1850 50  0001 C CNN
-	1    3000 1850
+P 3100 1350
+F 0 "#PWR015" H 3100 1100 50  0001 C CNN
+F 1 "Earth" H 3100 1200 50  0001 C CNN
+F 2 "" H 3100 1350 50  0001 C CNN
+F 3 "" H 3100 1350 50  0001 C CNN
+	1    3100 1350
 	1    0    0    -1
 $EndComp
@@
 L LM2936-3.3 U1
 U 1 1 5A02514F
-P 3400 1450
-F 0 "U1" H 3250 1575 50  0000 C CNN
-F 1 "LM3940" H 3400 1575 50  0000 L CNN
-F 2 "TO_SOT_Packages_SMD:SOT-223-3Lead_TabPin2" H 3400 1675 50  0001 C CIN
-F 3 "" H 3400 1400 50  0001 C CNN
-	1    3400 1450
+P 3500 950
+F 0 "U1" H 3350 1075 50  0000 C CNN
+F 1 "LM3940" H 3500 1075 50  0000 L CNN
+F 2 "TO_SOT_Packages_SMD:SOT-223-3Lead_TabPin2" H 3500 1175 50  0001 C CIN
+F 3 "" H 3500 900 50  0001 C CNN
+	1    3500 950
 	1    0    0    -1
 $EndComp
@@
 L Polyfuse_Small F2
 U 1 1 5A1493BC
-P 2800 1450
-F 0 "F2" V 2725 1450 50  0000 C CNN
-F 1 "0.5A" V 2875 1450 50  0000 C CNN
-F 2 "Fuse_Holders_and_Fuses:Fuse_SMD1206_Reflow" H 2850 1250 50  0001 L CNN
-F 3 "" H 2800 1450 50  0001 C CNN
-	1    2800 1450
+P 2900 950
+F 0 "F2" V 2825 950 50  0000 C CNN
+F 1 "0.5A" V 2975 950 50  0000 C CNN
+F 2 "Fuse_Holders_and_Fuses:Fuse_SMD1206_Reflow" H 2950 750 50  0001 L CNN
+F 3 "" H 2900 950 50  0001 C CNN
+	1    2900 950
 	0    -1   -1   0
 $EndComp
 Text Label 900  1350 0    40   ~ 0
 SUP_PROT
-Text Label 2900 1450 0    40   ~ 0
+Text Label 3000 950  0    40   ~ 0
 5V_PROT
 Text Label 1950 3000 1    40   ~ 0
@@
 F 0 "SW1" H 9100 1450 50  0000 L CNN
 F 1 "RESET" H 9050 1290 50  0000 C CNN
-F 2 "Buttons_Switches_SMD:SW_SPST_REED_CT05-XXXX-G1" H 9050 1550 50  0001 C CNN
+F 2 "Buttons_Switches_SMD:SW_SPST_SKQG" H 9050 1550 50  0001 C CNN
 F 3 "" H 9050 1550 50  0001 C CNN
 	1    9050 1350
@@
 Text Label 8400 1150 0    40   ~ 0
 OSCIN
-Text Label 6000 1600 1    40   ~ 0
+Text Label 6000 1750 1    40   ~ 0
 BOOT0
 Text Label 6100 1750 1    40   ~ 0
@@
 L LED_Small LED5
 U 1 1 5A1AF5A5
-P 4100 1850
-F 0 "LED5" H 4050 1975 50  0000 L CNN
-F 1 "RED" H 4000 1750 50  0000 L CNN
-F 2 "LEDs:LED_0603" V 4100 1850 50  0001 C CNN
-F 3 "" V 4100 1850 50  0001 C CNN
-	1    4100 1850
+P 4200 1350
+F 0 "LED5" H 4100 1450 50  0000 L CNN
+F 1 "RED" H 4100 1250 50  0000 L CNN
+F 2 "LEDs:LED_0603" V 4200 1350 50  0001 C CNN
+F 3 "" V 4200 1350 50  0001 C CNN
+	1    4200 1350
 	0    -1   -1   0
 $EndComp
@@
 L R_Small R3
 U 1 1 5A1AF662
-P 4100 1600
-F 0 "R3" H 4130 1620 50  0000 L CNN
-F 1 "520" H 4130 1560 50  0000 L CNN
-F 2 "Resistors_SMD:R_0805" H 4100 1600 50  0001 C CNN
-F 3 "" H 4100 1600 50  0001 C CNN
-	1    4100 1600
+P 4200 1100
+F 0 "R3" H 4230 1120 50  0000 L CNN
+F 1 "520" H 4230 1060 50  0000 L CNN
+F 2 "Resistors_SMD:R_0805" H 4200 1100 50  0001 C CNN
+F 3 "" H 4200 1100 50  0001 C CNN
+	1    4200 1100
 	1    0    0    -1
 $EndComp
@@
 L Earth #PWR019
 U 1 1 5A1B01CE
-P 4100 2050
-F 0 "#PWR019" H 4100 1800 50  0001 C CNN
-F 1 "Earth" H 4100 1900 50  0001 C CNN
-F 2 "" H 4100 2050 50  0001 C CNN
-F 3 "" H 4100 2050 50  0001 C CNN
-	1    4100 2050
+P 4200 1550
+F 0 "#PWR019" H 4200 1300 50  0001 C CNN
+F 1 "Earth" H 4200 1400 50  0001 C CNN
+F 2 "" H 4200 1550 50  0001 C CNN
+F 3 "" H 4200 1550 50  0001 C CNN
+	1    4200 1550
 	1    0    0    -1
 $EndComp
@@
 	2550 1450 2700 1450
 Wire Wire Line
-	3400 1750 3400 1850
-Wire Wire Line
-	3700 1450 4250 1450
-Wire Wire Line
-	3750 1450 3750 1550
-Connection ~ 3750 1450
-Wire Wire Line
-	3750 1750 3750 1850
-Wire Wire Line
-	3000 1750 3000 1850
-Connection ~ 2650 1450
+	3500 1250 3500 1350
+Wire Wire Line
+	3800 950  4350 950
+Wire Wire Line
+	3850 950  3850 1050
+Connection ~ 3850 950
+Wire Wire Line
+	3850 1250 3850 1350
+Wire Wire Line
+	3100 1250 3100 1350
 Wire Wire Line
 	850  900  850  1000
 Wire Wire Line
-	2900 1450 3100 1450
-Wire Wire Line
-	3000 1550 3000 1450
-Connection ~ 3000 1450
-Wire Wire Line
-	2650 1200 2650 1450
+	3000 950  3200 950
+Wire Wire Line
+	3100 1050 3100 950
+Connection ~ 3100 950
 Wire Wire Line
 	5700 4200 5700 4400
@@
 Connection ~ 2550 7100
 Wire Wire Line
-	4100 1700 4100 1750
-Wire Wire Line
-	4100 1500 4100 1450
-Connection ~ 4100 1450
-Wire Wire Line
-	4100 1950 4100 2050
+	4200 1200 4200 1250
+Wire Wire Line
+	4200 1000 4200 950
+Connection ~ 4200 950
+Wire Wire Line
+	4200 1450 4200 1550
 Wire Wire Line
 	4900 2400 4400 2400
@@
 $EndComp
 $Comp
-L Earth #PWR?
+L Earth #PWR028
 U 1 1 5A76FDB7
 P 7400 5650
-F 0 "#PWR?" H 7400 5400 50  0001 C CNN
+F 0 "#PWR028" H 7400 5400 50  0001 C CNN
 F 1 "Earth" H 7400 5500 50  0001 C CNN
 F 2 "" H 7400 5650 50  0001 C CNN
@@
 Wire Wire Line
 	7400 5550 7400 5650
+$Comp
+L D_Schottky D2
+U 1 1 5A8351B0
+P 2700 1150
+F 0 "D2" H 2700 1250 50  0000 C CNN
+F 1 "SS14" H 2700 1050 50  0000 C CNN
+F 2 "Diodes_SMD:D_SMA_Standard" H 2700 1150 50  0001 C CNN
+F 3 "" H 2700 1150 50  0001 C CNN
+	1    2700 1150
+	0    1    1    0
+$EndComp
+Wire Wire Line
+	2700 1450 2700 1300
+Wire Wire Line
+	2700 1000 2700 950
+Wire Wire Line
+	2500 950  2800 950
+Connection ~ 2700 950
+$Comp
+L R_Small R19
+U 1 1 5A84820F
+P 10250 3000
+F 0 "R19" H 10280 3020 50  0000 L CNN
+F 1 "10K" H 10280 2960 50  0000 L CNN
+F 2 "Resistors_SMD:R_0805" H 10250 3000 50  0001 C CNN
+F 3 "" H 10250 3000 50  0001 C CNN
+	1    10250 3000
+	0    1    1    0
+$EndComp
+Wire Wire Line
+	10150 3000 9950 3000
+Text Label 9950 3000 0    40   ~ 0
+BOOT1
+$Comp
+L Earth #PWR029
+U 1 1 5A8485E8
+P 10450 3150
+F 0 "#PWR029" H 10450 2900 50  0001 C CNN
+F 1 "Earth" H 10450 3000 50  0001 C CNN
+F 2 "" H 10450 3150 50  0001 C CNN
+F 3 "" H 10450 3150 50  0001 C CNN
+	1    10450 3150
+	1    0    0    -1
+$EndComp
+Wire Wire Line
+	10350 3000 10450 3000
+Wire Wire Line
+	10450 3000 10450 3150
+Text Label 2700 1450 2    40   ~ 0
+5V_OUT
 $EndSCHEMATC

Commit message: Preparing release 0.7
Parts:
- C1: footprint Capacitors_ThroughHole:CP_Radial_D8.0mm_P3.80mm -> Capacitors_ThroughHole:CP_Radial_D6.3mm_P2.50mm
Connections:
- wire segments 177 -> 178
Changed lines of the file:
@@
 F 0 "C1" H 1375 1050 50  0000 L CNN
 F 1 "330uF" H 1375 850 50  0000 L CNN
-F 2 "Capacitors_ThroughHole:CP_Radial_D8.0mm_P3.80mm" H 1350 950 50  0001 C CNN
+F 2 "Capacitors_ThroughHole:CP_Radial_D6.3mm_P2.50mm" H 1350 950 50  0001 C CNN
 F 3 "" H 1350 950 50  0001 C CNN
 	1    1350 950
@@
 F3 "CON_OUTPUT" I L 8300 5900 60
 F4 "BT_PAIRED" O L 8300 5550 60
+F5 "RESET" I L 8300 6050 60
 $EndSheet
 Wire Wire Line
@@
 Text Label 2700 1450 2    40   ~ 0
 5V_OUT
+Wire Wire Line
+	7900 6050 8300 6050
+Text Label 7950 6050 0    40   ~ 0
+RESET
 $EndSCHEMATC
