File: hardware/kedtracker.sch (KiCad schematic (older format))
At the start: 52 parts, among them J1 ANT, J2 SWD, J3 BOOT, J8 VK2828U7G5LF, J9 SDCARD_READER, SW1 RESET, U1 LM3940, Y2 8M

Commit message: Update schematics to latest KiCAD version
Parts:
- B1: symbol BUCK_CVTR -> kedtracker-rescue:BUCK_CVTR
- B2: symbol BMP280 -> kedtracker-rescue:BMP280
- C1: symbol CP1 -> kedtracker-rescue:CP1
- C10, C11, C14, C15, C16, C17, C18, C2, C3, C4, C5, C6, C7, C8, C9: symbol C_Small -> kedtracker-rescue:C_Small
- D1: symbol D -> kedtracker-rescue:D
- D2: symbol D_Schottky -> kedtracker-rescue:D_Schottky
- F1, F2: symbol Polyfuse_Small -> kedtracker-rescue:Polyfuse_Small
- J1: symbol CONN_COAXIAL -> kedtracker-rescue:CONN_COAXIAL
- J2: symbol CONN_01X04 -> kedtracker-rescue:CONN_01X04
- J3: symbol CONN_01X02 -> kedtracker-rescue:CONN_01X02
- J8: symbol VK2828U7G5LF -> kedtracker-rescue:VK2828U7G5LF
- J9: symbol Micro_SD_Card_Det1 -> kedtracker-rescue:Micro_SD_Card_Det1
- L1: symbol Ferrite_Bead -> kedtracker-rescue:Ferrite_Bead
- LED1, LED2, LED5: symbol LED_Small -> kedtracker-rescue:LED_Small
- LED3: symbol LED -> kedtracker-rescue:LED
- LS1: symbol Speaker -> kedtracker-rescue:Speaker
- MCU1: symbol STM32F103 -> kedtracker-rescue:STM32F103
- R1, R11, R12, R13, R19, R2, R3, R4, R5, R6, R7, R8: symbol R_Small -> kedtracker-rescue:R_Small
- R10, R9: symbol R -> kedtracker-rescue:R
- RF1: symbol RFM69HW -> kedtracker-rescue:RFM69HW
- SW1: symbol SW_Push -> kedtracker-rescue:SW_Push
- U1: symbol LM2936-3.3 -> kedtracker-rescue:LM2936-3.3
- Y2: symbol Crystal_Small -> kedtracker-rescue:Crystal_Small
Connections:
- wire segments 178 -> 220
